File: KiCad/STM32_Breakout.sch (KiCad schematic (older format))
At the start: 17 parts, among them J1 USB_B_Micro, J2 Conn_01x02, J3 Conn_01x12, J4 Conn_01x12, U1 STM32F042F6Px, U2 AP2127K-3.3

Commit message: save unsaved changes
Parts:
- renumbered BOOT to RST1
Connections:
- net PA5: now also R2.1
- net PB1: no longer R2.1
Changed lines of the file:
@@
 $EndComp
 $Comp
-L STM32_Breakout:SW_SPST BOOT
+L STM32_Breakout:SW_SPST RST1
 U 1 1 5FDE89BD
 P 5300 1450
-F 0 "BOOT" H 5300 1685 50  0000 C CNN
+F 0 "RST1" H 5300 1685 50  0000 C CNN
 F 1 "SW_SPST" H 5300 1594 50  0000 C CNN
 F 2 "STM32_Breakout:2PinTactileButton" H 5300 1450 50  0001 C CNN
@@
 	3850 4100 3850 4000
 Text GLabel 3750 4000 0    50   Input ~ 0
-PB1
+PA5
 Wire Wire Line
 	3750 4000 3850 4000
