File: KiCad/STM32_Breakout.kicad_pcb (KiCad board)
At the start: 2 copper layers, 15.2 x 33 mm, 17 parts, among them J1 USB_B_Micro, J2 Conn_01x02, J3 Conn_01x12, J4 Conn_01x12, U1 STM32F042F6Px, U2 AP2127K-3.3

Commit message: save unsaved changes
Parts:
- added G***: LOGO, TRA_KiCad_Footprints:VoronLogo_6pt5mm_silkScreen, B.Cu at (128.1, 76.1)
- added G***: LOGO, STM32_Breakout:THeyMadeME, F.Cu at (128.3, 90.2)
- renumbered BOOT1 to RST

Commit message: Update pin
Other:
- board text added: "+5V"
Changed lines of the file:
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@@
     (add_net "Net-(D1-Pad2)")
     (add_net "Net-(D2-Pad2)")
-    (add_net "Net-(U2-Pad4)")
     (add_net PA0)
     (add_net PA1)
@@
     )
   )
+  (dimension 12.7 (width 0.11) (layer Eco2.User)
+    (gr_text "12.700 mm" (at 128.27 69.312001) (layer Eco2.User)
+      (effects (font (size 1 1) (thickness 0.15)))
+    )
+    (feature1 (pts (xy 121.92 76.2) (xy 121.92 70.02558)))
+    (feature2 (pts (xy 134.62 76.2) (xy 134.62 70.02558)))
+    (crossbar (pts (xy 134.62 70.612001) (xy 121.92 70.612001)))
+    (arrow1a (pts (xy 121.92 70.612001) (xy 123.046504 70.02558)))
+    (arrow1b (pts (xy 121.92 70.612001) (xy 123.046504 71.198422)))
+    (arrow2a (pts (xy 134.62 70.612001) (xy 133.493496 70.02558)))
+    (arrow2b (pts (xy 134.62 70.612001) (xy 133.493496 71.198422)))
+  )
   (dimension 33.02 (width 0.15) (layer Eco2.User)
     (gr_text "33.020 mm" (at 147.223 88.9 270) (layer Eco2.User)
@@
     (effects (font (size 0.8 0.8) (thickness 0.15)))
   )
-  (gr_text GND (at 122.174 74.422 15) (layer F.SilkS)
+  (gr_text +5V (at 122.174 74.422 15) (layer F.SilkS)
     (effects (font (size 0.8 0.8) (thickness 0.15)))
   )
@@
   (gr_text PA3 (at 133.12 99.06 105) (layer F.SilkS)
     (effects (font (size 0.8 0.8) (thickness 0.15)))
-  )
-  (dimension 12.7 (width 0.11) (layer Eco2.User)
-    (gr_text "12.700 mm" (at 128.27 69.312001) (layer Eco2.User)
-      (effects (font (size 1 1) (thickness 0.15)))
-    )
-    (feature1 (pts (xy 121.92 76.2) (xy 121.92 70.02558)))
-    (feature2 (pts (xy 134.62 76.2) (xy 134.62 70.02558)))
-    (crossbar (pts (xy 134.62 70.612001) (xy 121.92 70.612001)))
-    (arrow1a (pts (xy 121.92 70.612001) (xy 123.046504 70.02558)))
-    (arrow1b (pts (xy 121.92 70.612001) (xy 123.046504 71.198422)))
-    (arrow2a (pts (xy 134.62 70.612001) (xy 133.493496 70.02558)))
-    (arrow2b (pts (xy 134.62 70.612001) (xy 133.493496 71.198422)))
   )
   (gr_line (start 128.27 74.93) (end 128.27 105.41) (layer Eco2.User) (width 0.15))
@@
     (connect_pads (clearance 0.3))
     (min_thickness 0.254)
-    (fill yes (arc_segments 32) (thermal_gap 0.508) (thermal_bridge_width 0.508))
+    (fill (arc_segments 32) (thermal_gap 0.508) (thermal_bridge_width 0.508))
     (polygon
       (pts
@@
     (connect_pads (clearance 0.3))
     (min_thickness 0.254)
-    (fill yes (arc_segments 32) (thermal_gap 0.508) (thermal_bridge_width 0.508))
+    (fill (arc_segments 32) (thermal_gap 0.508) (thermal_bridge_width 0.508))
     (polygon
       (pts
