File: KiCad/STM32_Breakout.kicad_pcb (KiCad board)
At the start: 2 copper layers, 15.2 x 33 mm, 17 parts, among them J1 USB_B_Micro, J2 Conn_01x02, J3 Conn_01x12, J4 Conn_01x12, U1 STM32F042F6Px, U2 AP2127K-3.3

Commit message: Patch 002 (#1)
* add ignore

* Clean up ignored files

* save unsaved changes

* Update pin
Parts:
- added G***: LOGO, TRA_KiCad_Footprints:VoronLogo_6pt5mm_silkScreen, B.Cu at (128.1, 76.1)
- added G***: LOGO, STM32_Breakout:THeyMadeME, F.Cu at (128.3, 90.2)
- renumbered BOOT1 to RST
Other:
- board text added: "+5V"
